File: CSI DPT/CSI_DPT.kicad_pcb (KiCad board)
At the start: 4 copper layers, 100 x 80 mm, 49 parts, among them J3 SSW-102-01-G-D, J4 Conn_02x08_Odd_Even, Q1 DMP3099L, U1 UCC23513QDWYRQ1, U2 MGJ2D121802SC, U4 LDK130-12_SOT23_SOT353, U5 NC7SZ125M5X, U7 ADM4168EBRUZ, U8 MGJ2D121802SC, U9 LT1086-ADJ

Commit message: Nov.18 Update 1
temp
Parts:
- removed MH1, MH2, MH3: MountingHole_4.3mm_M4_DIN965, MountingHole:MountingHole_4.3mm_M4_DIN965
- moved PWM_H 51.3 mm to (125.8, 91.6)
- renumbered TP8 to PWM_H, VIN12V to TP1, GND1 to TP2, VIN5V to TP3, GND1 to TP4, 1.2V to TP5, 0V to TP6, -18V to TP7
Connections:
- U7 pad 12: /Gate_Driver/0V -> GND1
- U7 pad 4: /Gate_Driver/0V -> GND1
Routing:
- net GND1: track 94.3 -> 102.6 mm, vias 4 -> 5

Commit message: Nov.18 Update 2
1. Finish PCB layout
Parts:
- added H1: MountingHole, MountingHole:MountingHole_4.3mm_M4_DIN965, F.Cu at (161.6, 101.9)
- added H2: MountingHole, MountingHole:MountingHole_4.3mm_M4_DIN965, F.Cu at (92.0, 67.4)
- added H3: MountingHole, MountingHole:MountingHole_4.3mm_M4_DIN965, F.Cu at (92.0, 136.5)
- moved LS_P1 127.1 mm to (69.1, 134.0)
- moved LS_N1 125.2 mm to (69.2, 138.8)
- moved HS_P1 107.7 mm to (68.8, 65.0)
- moved HS_N1 107.7 mm to (68.8, 69.5)
- moved VGATE_H1 11.6 mm to (161.6, 70.1)
- moved 0V1 11.0 mm to (161.7, 75.9)
- moved PWM_H1 10.4 mm to (115.6, 89.6)
- renumbered TP7 to -18V1, TP10 to 0V1, TP6 to 0V2, TP5 to 1.2V1, TP2 to GND1A1, TP4 to GND1B1, TP13 to HS_N1, TP11 to HS_P1, TP14 to LS_N1, TP12 to LS_P1, PWM_H to PWM_H1, TP9 to VGATE_H1, TP1 to VIN12V1, TP3 to VIN5V1
Connections:
- net Net-(J3-Pad1) renamed /Gate_Driver/VGATE_H
- HS_N1 pad 1: unconnected-(TP13-Pad1) -> /Gate_Driver/HS_N
- HS_P1 pad 1: unconnected-(TP11-Pad1) -> /Gate_Driver/HS_P
- LS_N1 pad 1: unconnected-(TP14-Pad1) -> /Gate_Driver/LS_N
- LS_P1 pad 1: unconnected-(TP12-Pad1) -> /Gate_Driver/LS_P
Routing:
- net /Gate_Driver/LS_N: track 27.9 -> 74.5 mm, vias 0 -> 1
- net /Gate_Driver/LS_P: track 31.1 -> 70.6 mm, vias 0 -> 1
- net /Gate_Driver/HS_P: track 32.0 -> 63.1 mm, vias 2 -> 3
- net /Gate_Driver/HS_N: track 27.3 -> 58.0 mm, vias 0 -> 1
- net /Gate_Driver/VGATE_H: track 6.50 -> 21.6 mm, vias 0 -> 1
- net /Gate_Driver/0V: track 76.1 -> 67.4 mm, vias 0 -> 4
- net /Gate_Driver/-18V: track 44.8 -> 51.7 mm, vias 1 -> 2
- net /Gate_Driver/PWM_H: track 28.9 -> 34.3 mm, vias 0 -> 1
- net GND1: track 102.6 -> 106.3 mm
- added copper zone on In1.Cu, net /Gate_Driver/-18V
- added copper zone on In1.Cu, net /Gate_Driver/0V
