File: CSI DPT/CSI_DPT.kicad_pcb (KiCad board)
At the start: 4 copper layers, 100 x 80 mm, 49 parts, among them J3 SSW-102-01-G-D, J4 Conn_02x08_Odd_Even, Q1 DMP3099L, U1 UCC23513QDWYRQ1, U2 MGJ2D121802SC, U4 LDK130-12_SOT23_SOT353, U5 NC7SZ125M5X, U7 ADM4168EBRUZ, U8 MGJ2D121802SC, U9 LT1086-ADJ

Commit message: test commit
Parts:
- renumbered J4 to J2, Q1 to Q3
Connections:
- net /Gate_Driver/-18V renamed /Gate_Driver/-18V_H
- net /Gate_Driver/1.2V renamed /Gate_Driver/1.2V_H
- 0V2 pad 1: /Gate_Driver/0V -> /Gate_Driver/0V_H
- C1 pad 2: /Gate_Driver/0V -> /Gate_Driver/0V_H
- C2 pad 2: /Gate_Driver/0V -> /Gate_Driver/0V_H
- C3 pad 2: /Gate_Driver/0V -> /Gate_Driver/0V_H
- C4 pad 2: /Gate_Driver/0V -> /Gate_Driver/0V_H
- C5 pad 2: /Gate_Driver/0V -> /Gate_Driver/0V_H
- C6 pad 1: /Gate_Driver/0V -> /Gate_Driver/0V_H
- C7 pad 1: /Gate_Driver/0V -> /Gate_Driver/0V_H
- C8 pad 1: /Gate_Driver/0V -> /Gate_Driver/0V_H
- C9 pad 1: /Gate_Driver/0V -> /Gate_Driver/0V_H
- U2 pad 7: /Gate_Driver/0V -> /Gate_Driver/0V_H
- U4 pad 2: /Gate_Driver/0V -> /Gate_Driver/0V_H
- U8 pad 5: /Gate_Driver/0V -> /Gate_Driver/0V_H
Routing:
- net /Gate_Driver/0V_H: track 0.00 -> 52.1 mm
- net /Gate_Driver/0V: track 67.4 -> 15.3 mm
