File: CSI DPT/Tester_Board.kicad_sch (KiCad schematic)
At the start: 0 parts

Commit message: test commit
Parts:
- added D1, D2: UJ3N065025K3S, Package_TO_SOT_THT:TO-247-2_Vertical, symbol Device:D_Schottky
- added H4, H5, H6, H7: MountingHole, MountingHole:MountingHole_4.3mm_M4_DIN965, symbol Mechanical:MountingHole
- added Q1, Q2: UJ3N065025K3S, Package_TO_SOT_THT:TO-247-3_Vertical, symbol UJ3N065025K3S:UJ3N065025K3S
Connections:
- new net: D2.2 (A), Q2.3 (S)
- new net: D1.2 (A), Q1.3 (S)
